Commit message: fix: rename package
Signed-off-by: Maciej Krupka <maciej.p.krupka@student.put.poznan.pl>

File: unitree_a1_description/xacro/gazebo.xacro (robot description, xacro)
@@ -4,5 +4,5 @@
     <gazebo>
         <plugin filename="libgazebo_ros2_control.so" name="gazebo_ros2_control">
-            <parameters>$(find a1_description)/config/robot_controller.yaml</parameters>
+            <parameters>$(find unitree_a1_description)/config/robot_controller.yaml</parameters>
         </plugin>
     </gazebo>

File: unitree_a1_description/xacro/leg.xacro (robot description, xacro)
@@ -1,5 +1,5 @@
 <?xml version="1.0"?>
 <robot xmlns:xacro="http://www.ros.org/wiki/xacro">
-    <xacro:include filename="$(find a1_description)/xacro/transmission.xacro"/>
+    <xacro:include filename="$(find unitree_a1_description)/xacro/transmission.xacro"/>
     <xacro:macro name="leg" params="name mirror mirror_dae front_hind front_hind_dae *origin">
         <joint name="${name}_hip_joint" type="revolute">
@@ -31,5 +31,5 @@
                 </xacro:if>
                 <geometry>
-                    <mesh filename="file://$(find a1_description)/meshes/hip.dae" scale="1 1 1"/>
+                    <mesh filename="file://$(find unitree_a1_description)/meshes/hip.dae" scale="1 1 1"/>
                 </geometry>
                 <material name="orange"/>
@@ -77,8 +77,8 @@
                 <geometry>
                     <xacro:if value="${mirror_dae == True}">
-                        <mesh filename="file://$(find a1_description)/meshes/thigh.dae" scale="1 1 1"/>
+                        <mesh filename="file://$(find unitree_a1_description)/meshes/thigh.dae" scale="1 1 1"/>
                     </xacro:if>
                     <xacro:if value="${mirror_dae == False}">
-                        <mesh filename="file://$(find a1_description)/meshes/thigh_mirror.dae" scale="1 1 1"/>
+                        <mesh filename="file://$(find unitree_a1_description)/meshes/thigh_mirror.dae" scale="1 1 1"/>
                     </xacro:if>
                 </geometry>
@@ -112,5 +112,5 @@
                 <origin rpy="0 0 0" xyz="0 0 0"/>
                 <geometry>
-                    <mesh filename="file://$(find a1_description)/meshes/calf.dae" scale="1 1 1"/>
+                    <mesh filename="file://$(find unitree_a1_description)/meshes/calf.dae" scale="1 1 1"/>
                 </geometry>
                 <material name="orange"/>

File: unitree_a1_description/xacro/robot.xacro (robot description, xacro)
@@ -2,10 +2,10 @@
 <robot name="a1" xmlns:xacro="http://www.ros.org/wiki/xacro">
     <xacro:arg name="DEBUG" default="false"/>
-    <xacro:include filename="$(find a1_description)/xacro/const.xacro"/>
-    <xacro:include filename="$(find a1_description)/xacro/materials.xacro"/>
-    <xacro:include filename="$(find a1_description)/xacro/leg.xacro"/>
+    <xacro:include filename="$(find unitree_a1_description)/xacro/const.xacro"/>
+    <xacro:include filename="$(find unitree_a1_description)/xacro/materials.xacro"/>
+    <xacro:include filename="$(find unitree_a1_description)/xacro/leg.xacro"/>
     <!-- <xacro:include filename="$(find a1_description)/xacro/stairs.xacro"/> -->
-    <xacro:include filename="$(find a1_description)/xacro/gazebo.xacro"/>
-    <xacro:include filename="$(find a1_description)/xacro/ros2_control.xacro"/>
+    <xacro:include filename="$(find unitree_a1_description)/xacro/gazebo.xacro"/>
+    <xacro:include filename="$(find unitree_a1_description)/xacro/ros2_control.xacro"/>
     <!-- <xacro:include filename="$(find a1_gazebo)/launch/stairs.urdf.xacro"/> -->
     <!-- <xacro:stairs stairs="15" xpos="0" ypos="0" zpos="0" /> -->
@@ -38,5 +38,5 @@
             <origin rpy="0 0 0" xyz="0 0 0"/>
             <geometry>
-                <mesh filename="file://$(find a1_description)/meshes/trunk.dae" scale="1 1 1"/>
+                <mesh filename="file://$(find unitree_a1_description)/meshes/trunk.dae" scale="1 1 1"/>
             </geometry>
             <material name="orange"/>
