Commit message: fix: urdf
Signed-off-by: Maciej Krupka <maciej.p.krupka@student.put.poznan.pl>

File: unitree_a1_description/urdf/a1.urdf (robot description, URDF)
Before this commit: robot a1, 23 links, 22 joints
Links:
- link FL_calf: geometry collision box size=0.2 0.016 0.016; visual mesh filename=package://unitree_a1_description/meshes/calf.dae scale=1 1 1
- link FL_hip: geometry collision cylinder length=0.04 radius=0.046; visual mesh filename=package://unitree_a1_description/meshes/hip.dae scale=1 1 1
- link FL_thigh: geometry collision box size=0.2 0.0245 0.034; visual mesh filename=package://unitree_a1_description/meshes/thigh.dae scale=1 1 1
- link FR_calf: geometry collision box size=0.2 0.016 0.016; visual mesh filename=package://unitree_a1_description/meshes/calf.dae scale=1 1 1
- link FR_hip: geometry collision cylinder length=0.04 radius=0.046; visual mesh filename=package://unitree_a1_description/meshes/hip.dae scale=1 1 1
- link FR_thigh: geometry collision box size=0.2 0.0245 0.034; visual mesh filename=package://unitree_a1_description/meshes/thigh_mirror.dae scale=1 1 1
- link RL_calf: geometry collision box size=0.2 0.016 0.016; visual mesh filename=package://unitree_a1_description/meshes/calf.dae scale=1 1 1
- link RL_hip: geometry collision cylinder length=0.04 radius=0.046; visual mesh filename=package://unitree_a1_description/meshes/hip.dae scale=1 1 1
- link RL_thigh: geometry collision box size=0.2 0.0245 0.034; visual mesh filename=package://unitree_a1_description/meshes/thigh.dae scale=1 1 1
- link RR_calf: geometry collision box size=0.2 0.016 0.016; visual mesh filename=package://unitree_a1_description/meshes/calf.dae scale=1 1 1
- link RR_hip: geometry collision cylinder length=0.04 radius=0.046; visual mesh filename=package://unitree_a1_description/meshes/hip.dae scale=1 1 1
- link RR_thigh: geometry collision box size=0.2 0.0245 0.034; visual mesh filename=package://unitree_a1_description/meshes/thigh_mirror.dae scale=1 1 1
- link trunk: geometry collision box size=0.267 0.194 0.114; visual mesh filename=package://unitree_a1_description/meshes/trunk.dae scale=1 1 1

File: unitree_a1_description/xacro/robot.xacro (robot description, xacro)
@@ -5,5 +5,5 @@
     <xacro:include filename="$(find unitree_a1_description)/xacro/materials.xacro"/>
     <xacro:include filename="$(find unitree_a1_description)/xacro/leg.xacro"/>
-    <!-- <xacro:include filename="$(find a1_description)/xacro/stairs.xacro"/> -->
+    <!-- <xacro:include filename="$(find unitree_a1_description)/xacro/stairs.xacro"/> -->
     <xacro:include filename="$(find unitree_a1_description)/xacro/gazebo.xacro"/>
     <xacro:include filename="$(find unitree_a1_description)/xacro/ros2_control.xacro"/>
